File: a500hdd.sch (KiCad schematic (older format))
At the start: 28 parts, among them U1 ata_connector, U3 74LS04, U4 a500exp, U5 74LS00, U6 74LS08, U7 74LS08

Commit message: Added ATA44 header to schematic
Parts:
- added R18: 4k7, Resistors_SMD:R_0805, symbol R
- added U2: ata_connector44, Pin_Headers:Pin_Header_Straight_2x22_Pitch2.00mm, symbol ata_connector44
Connections:
- net labels added: DATA, ENABLE, ~ATA_ACTILED, ~ATA_RESET
- net labels removed: ACTLED, ADDREN, AS, ATA_D0, ATA_D1, ATA_D10, ATA_D11, ATA_D12, ATA_D13, ATA_D14, ATA_D15, ATA_D2, ATA_D3, ATA_D4, ATA_D5, ATA_D6, ATA_D7, ATA_D8, ATA_D9, ~ACTLED, ~RESET
- wire segments 151 -> 135
- no-connect marks 48 -> 55
Other:
- note added: "ATA Enable"
- note added: "ATA Read/Write"
- note added: "ATA40"
- note added: "ATA44"
- note added: "Activity LED"
- note added: "Decoupling"
- note added: "U3, U5, U6, U7"

Commit message: Rev2 PCB, migrated do KiCad5
Parts:
- removed U3: 74LS04, Housings_SOIC:SOIC-14_3.9x8.7mm_Pitch1.27mm, symbol 74LS04
- removed U5: 74LS00, Housings_SOIC:SOIC-14_3.9x8.7mm_Pitch1.27mm, symbol 74LS00
- removed U6, U7: 74LS08, Housings_SOIC:SOIC-14_3.9x8.7mm_Pitch1.27mm, symbol 74LS08
- added J1: Conn_01x04_Male, Connector_JST:JST_XH_S04B-XH-A_1x04_P2.50mm_Horizontal, symbol Connector:Conn_01x04_Male
- added JP1, JP2: SolderJumper_2_Bridged, Jumper:SolderJumper-2_P1.3mm_Open_Pad1.0x1.5mm, symbol Jumper:SolderJumper_2_Bridged
- added U3: 74LS04, Package_SO:SOIC-14_3.9x8.7mm_P1.27mm, symbol 74xx:74LS04
- added U5: 74LS00, Package_SO:SOIC-14_3.9x8.7mm_P1.27mm, symbol 74xx:74LS00
- added U6, U7: 74LS08, Package_SO:SOIC-14_3.9x8.7mm_P1.27mm, symbol 74xx:74LS08
- added U8: a500exp, a500hdd:header2x43, symbol a500hdd:a500exp
- added U9: a500exp, a500hdd:A500_Expansion_slot, symbol a500hdd:a500exp
- C1, C2, C3, C4: footprint Capacitors_SMD:C_0805 -> Capacitor_SMD:C_0805_2012Metric; symbol C -> Device:C
- D1: footprint LEDs:LED_0805 -> LED_SMD:LED_0805_2012Metric; symbol LED -> Device:LED
- R1, R10, R11, R12, R13, R14, R15, R16, R17, R18, R2, R3, R4, R5, R6, R7, R8, R9: footprint Resistors_SMD:R_0805 -> Capacitor_SMD:C_0805_2012Metric; symbol R -> Device:R
- U1: footprint Connect:IDC_Header_Straight_40pins -> Connector_IDC:IDC-Header_2x20_P2.54mm_Vertical; symbol ata_connector -> a500hdd:ata_connector
- U2: footprint Pin_Headers:Pin_Header_Straight_2x22_Pitch2.00mm -> Connector_PinSocket_2.00mm:PinSocket_2x22_P2.00mm_Vertical; symbol ata_connector44 -> a500hdd:ata_connector44
- U4: symbol a500exp -> a500hdd:a500exp
Connections:
- net labels added: +12V, B11, B46, B48, B50, B51, B53, B55, B60, B61, B62, B63, B64, B65, B66, B67, B68, B69, B7, B70, B71, B72, B73, B74, B75, B76, B77, B78, B79, B80, B81, B82, B83, B84, B85, B86, B9, ~ATA_CSA, ~ATA_CSB
- wire segments 135 -> 240
- no-connect marks 55 -> 54
Other:
- note added: "(optional)"
- note added: "Expansion port adapter"
- note added: "IDE Power"
- note added: "~CS~ swap"
